File: Scematics/MainBoard.sch (KiCad schematic (older format))
At the start: 35 parts

Commit message: Verbesserungen des Systemes
Parts:
- removed D? (x2): D, symbol D
- removed P? (x8): CONN_02X05, symbol CONN_02X05
- removed Q?: Q_PMOS_GSD, symbol Q_PMOS_GSD
- removed R?: R, symbol R
- removed SH?: TPIC6B595, symbol TPIC6B595
- added D2, D3, D4, D5, D6, D7, D8, D9: ON, symbol Led_Small
- added P2: CONN_02X08, symbol CONN_02X08
- added Q11, Q13, Q15, Q17, Q19, Q3, Q6, Q9: IRF510, TO_SOT_Packages_THT:TO-220_Neutral123_Vertical, symbol Q_NMOS_GDS
- added Q4: Q_NMOS_SGD, symbol Q_NMOS_SGD
- added Q7: Q_NMOS_GDS, symbol Q_NMOS_GDS
- added R1, R11, R13, R15, R17, R19, R2, R21, R5, R6, R8, R9: R, symbol R
- added U1: 74HC595, symbol 74HC595
- gave numbers to parts that had none: 22
Connections:
- net +5V: now also R1.1, U1.16 (VCC)
- net +BATT: now also Q10.3 (D), Q12.3 (D), Q14.3 (D), Q16.3 (D), Q18.3 (D), Q2.3 (D), Q5.3 (D), Q8.3 (D), R10.1, R12.1, R14.1, R16.1, R18.1, R20.1, R4.1, R7.1
- net FIRE: now also Q7.1 (G), R9.1
- net GND: now also Q4.1 (S), Q7.3 (S), R2.2, R6.2, R9.2, U1.8 (GND)
- net N0: now also P2.2 (P2), Q3.2 (D)
- net N1: now also P2.4 (P4), Q6.2 (D)
- net N2: now also P2.6 (P6), Q9.2 (D)
- net N3: now also P2.8 (P8), Q11.2 (D)
- net N4: now also P2.10 (P10), Q13.2 (D)
- net N5: now also P2.12 (P12), Q15.2 (D)
- net N6: now also P2.14 (P14), Q17.2 (D)
- net N7: now also P2.16 (P16), Q19.2 (D)
- net P0: now also P2.1 (P1)
- net P1: now also P2.3 (P3)
- net P2: now also P2.5 (P5)
- net P3: now also P2.7 (P7)
- net P4: now also P2.9 (P9)
- net P5: now also P2.11 (P11)
- net P6: now also P2.13 (P13)
- net P7: now also P2.15 (P15)
- net RCK: now also SH1.12 (RCK)
- net SER_IN: now also U1.12 (RCLK), U1.14 (SER)
- net SIGTAP: now also Q4.3 (D)
- net SRCK: now also SH1.13 (SRCK), U1.11 (SRCLK)
- net at SH1.3 (SER_IN): now also U1.9 (~QH)
- net SRCLR: now reaches SH1.8 (SRCLR)
- net SRCLR: now also R1.2, U1.10 (SRCLR)
- net EN: now reaches SH1.9 (EN)
- net EN: now also R2.1, U1.13 (G)
- net BRB: no longer names the net of P1.9 (P9)
- new net: D2.1 (K), D3.1 (K), D4.1 (K), D5.1 (K), D6.1 (K), D7.1 (K), D8.1 (K), D9.1 (K), Q11.3 (S), Q13.3 (S), Q15.3 (S), Q17.3 (S), Q19.3 (S), Q3.3 (S), Q4.2 (G), Q6.3 (S), Q7.2 (D), Q9.3 (S), R6.1
- new net: D2.2 (A), R5.2
- new net: D3.2 (A), R8.2
- new net: D4.2 (A), R11.2
- new net: D5.2 (A), R13.2
- new net: D6.2 (A), R15.2
- new net: D7.2 (A), R17.2
- new net: D8.2 (A), R19.2
- new net: D9.2 (A), R21.2
- new net NE0: Q3.1 (G), R5.1, U1.15 (QA)
- new net NE1: Q6.1 (G), R8.1, U1.1 (QB)
- new net NE2: Q9.1 (G), R11.1, U1.2 (QC)
- new net NE3: Q11.1 (G), R13.1, U1.3 (QD)
- new net NE4: Q13.1 (G), R15.1, U1.4 (QE)
- new net NE5: Q15.1 (G), R17.1, U1.5 (QF)
- new net NE6: Q17.1 (G), R19.1, U1.6 (QG)
- new net NE7: Q19.1 (G), R21.1, U1.7 (QH)
- no-connect marks 0 -> 5

Commit message: Changes to properly implement ON LEDs
Parts:
- removed D2, D3, D4, D5, D6, D7, D8, D9: ON, symbol Led_Small
- added D? (x16): ON, symbol Led_Small
- U1: symbol 74HC595 -> 74HC595-RESCUE-MainBoard
Connections:
- net NE0: now also D?.2 (A); no longer Q3.1 (G), R5.1
- net NE1: now also D?.2 (A); no longer Q6.1 (G), R8.1
- net NE2: now also D?.2 (A); no longer Q9.1 (G), R11.1
- net NE3: now also D?.2 (A); no longer Q11.1 (G), R13.1
- net NE4: now also D?.2 (A); no longer Q13.1 (G), R15.1
- net NE5: now also D?.2 (A); no longer Q15.1 (G), R17.1
- net NE6: now also D?.2 (A); no longer Q17.1 (G), R19.1
- net NE7: now also D?.2 (A); no longer Q19.1 (G), R21.1
- net PE0: now also D?.1 (K); no longer Q2.1 (G), R4.2
- net PE1: now also D?.1 (K); no longer Q5.1 (G), R7.2
- net PE2: now also D?.1 (K); no longer Q8.1 (G), R10.2
- net PE3: now also D?.1 (K); no longer Q10.1 (G), R12.2
- net PE4: now also D?.1 (K); no longer Q12.1 (G), R14.2
- net PE5: now also D?.1 (K); no longer Q14.1 (G), R16.2
- net PE6: now also D?.1 (K); no longer Q16.1 (G), R18.2
- net PE7: now also D?.1 (K); no longer Q18.1 (G), R20.2
- net at Q11.3 (S), Q13.3 (S), Q15.3 (S)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: now also R11.2, R13.2, R15.2, R17.2, R19.2, R21.2, R5.2, R8.2
- new net: D?.2 (A), Q2.1 (G), R4.2
- new net: D?.2 (A), Q5.1 (G), R7.2
- new net: D?.2 (A), Q8.1 (G), R10.2
- new net: D?.2 (A), Q10.1 (G), R12.2
- new net: D?.2 (A), Q12.1 (G), R14.2
- new net: D?.2 (A), Q14.1 (G), R16.2
- new net: D?.2 (A), Q16.1 (G), R18.2
- new net: D?.2 (A), Q18.1 (G), R20.2
- new net: D?.1 (K), Q3.1 (G), R5.1
- new net: D?.1 (K), Q6.1 (G), R8.1
- new net: D?.1 (K), Q9.1 (G), R11.1
- new net: D?.1 (K), Q11.1 (G), R13.1
- new net: D?.1 (K), Q13.1 (G), R15.1
- new net: D?.1 (K), Q15.1 (G), R17.1
- new net: D?.1 (K), Q17.1 (G), R19.1
- new net: D?.1 (K), Q19.1 (G), R21.1
