File: Scematics/ArduinoBoard/ArduinoBoard.sch (KiCad schematic (older format))
At the start: 11 parts

Commit message: Changes for real soldering
Connections:
- net P_ON is gone; now on net LOCK: P?.4 (P4)
- net +5V: now also P?.2 (P2); no longer P?.1 (P1)
- net BNT: now also P?.1 (P1); no longer P?.2 (P2)
Changed lines of the file:
@@
 	3100 2800 2850 2800
 Text Label 2850 2800 0    60   ~ 0
-P_ON
+LOCK
 Wire Wire Line
 	3100 2700 2850 2700
@@
 $EndComp
 $Comp
-L +5V #PWR?
-U 1 1 584EE04E
-P 4250 3900
-F 0 "#PWR?" H 4250 3750 50  0001 C CNN
-F 1 "+5V" H 4250 4040 50  0000 C CNN
-F 2 "" H 4250 3900 50  0000 C CNN
-F 3 "" H 4250 3900 50  0000 C CNN
-	1    4250 3900
-	1    0    0    -1
-$EndComp
-Wire Wire Line
-	4250 3900 4250 4000
-$Comp
 L Q_NMOS_DGS Q?
 U 1 1 584EE26B
@@
 	1    0    0    -1
 $EndComp
-Wire Wire Line
-	4000 4100 4250 4100
 $Comp
 L GND #PWR?
@@
 Text Label 4000 3650 0    60   ~ 0
 BNT
+Wire Wire Line
+	4000 4000 4250 4000
+Connection ~ 4000 4000
+$Comp
+L +5V #PWR?
+U 1 1 584EC22A
+P 4150 4200
+F 0 "#PWR?" H 4150 4050 50  0001 C CNN
+F 1 "+5V" H 4150 4340 50  0000 C CNN
+F 2 "" H 4150 4200 50  0000 C CNN
+F 3 "" H 4150 4200 50  0000 C CNN
+	1    4150 4200
+	1    0    0    -1
+$EndComp
+Wire Wire Line
+	4150 4200 4200 4200
+Wire Wire Line
+	4200 4200 4200 4100
+Wire Wire Line
+	4200 4100 4250 4100
 $EndSCHEMATC

Commit message: Tweaked the schematics a bit (version update)
Parts:
- BT?: symbol Battery -> Battery-RESCUE-ArduinoBoard
Other:
- note added: "PB3\nPB2\nPB1\nPB0"
- note added: "PD7\nPD6\nPD5\nPD4\nPD3\nPD2\nPD1\nPD0"
Changed lines of the file:
@@
 EESchema Schematic File Version 2
+LIBS:ArduinoBoard-rescue
 LIBS:power
 LIBS:device
@@
 $EndComp
 $Comp
-L Battery BT?
+L Battery-RESCUE-ArduinoBoard BT?
 U 1 1 584AEE68
 P 1850 4150
@@
 Wire Wire Line
 	4200 4100 4250 4100
+Text Notes 3450 2300 0    60   ~ 0
+PB3\nPB2\nPB1\nPB0
+Text Notes 3450 3200 0    60   ~ 0
+PD7\nPD6\nPD5\nPD4\nPD3\nPD2\nPD1\nPD0
 $EndSCHEMATC
