File: Scematics/MainBoard/MainBoard.sch (KiCad schematic (older format))
At the start: 62 parts, among them P1 CONN_02X05, P2 CONN_02X08, Q1 Q_NMOS_SGD, Q10 PMOS, Q11 IRF510, Q12 PMOS, Q13 IRF510, Q14 PMOS, Q15 IRF510, Q16 PMOS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

Commit message: Tweaked the schematics a bit (version update)
Parts:
- BT1: symbol Battery -> Battery-RESCUE-MainBoard
Changed lines of the file:
@@
 	3000 6100 2450 6100
 $Comp
-L Battery BT1
+L Battery-RESCUE-MainBoard BT1
 U 1 1 584704B3
 P 4000 6900
